File: Deliverable #3/Automatic Pet Feeder.sch (EAGLE design)
At the start: 62 parts, among them M1 SERVO, Q1 MMBT4403, Q2 MMBT4403, U1 JOYSTICKPTH, U2 HX711, U3 JOYSTICKPTH, U4 MSP430FR5994IZVW, U5 HX711, U6 VL6180V1NR/1, U7 OSHW-LOGOS

Commit message: Reworked schematic
Parts:
- removed C1, C10, C11, C12, C13, C14, C2, C3, C4, C5: 0.1uF, SparkFun-Capacitors:0.1UF-25V-5%(0603)
- removed C6, C7, C8, C9: 10uF, SparkFun-Capacitors:10UF50V20%(1210)
- removed FID1, FID2: FIDUCIAL1X2, SparkFun-Aesthetics:FIDUCIAL1X2
- removed FRAME1: FRAME-LETTER, SparkFun-Aesthetics:FRAME-LETTER
- removed J1, J2, JP4, JP6: (no value), SparkFun-Connectors:M05PTH
- removed JP1: (no value), pinhead:PINHD-1X5
- removed JP2, JP5: (no value), SparkFun-Connectors:M02PTH
- removed L1, L2: 3.3uH, SparkFun-Passives:INDUCTOR0805-IND
- removed LOGO1: SFE_LOGO_NAME_FLAME.1_INCH, SparkFun-Aesthetics:SFE_LOGO_NAME_FLAME.1_INCH
- removed LOGO3: SFE_LOGO_FLAME.1_INCH, SparkFun-Aesthetics:SFE_LOGO_FLAME.1_INCH
- removed Q1, Q2: MMBT4403, SparkFun-DiscreteSemi:TRANSISTOR_PNPMMBT4403
- removed R1, R9: 20k, SparkFun-Resistors:20KOHM1/10W1%(0603)
- removed R10, R5: 10K, SparkFun-Resistors:10KOHM-1/10W-1%(0603)0603
- removed R2, R8: 8.2K, SparkFun-Resistors:8.2KOHM-1/10W-5%(0603)
- removed R3, R4, R6, R7: 100, SparkFun-Resistors:100OHM-1/10W-1%(0603)
- removed SJ1, SJ2: JUMPER-PAD-2-NC_BY_TRACE, SparkFun-Passives:JUMPER-PAD-2-NC_BY_TRACE
- removed STANDOFF1, STANDOFF2, STANDOFF3, STANDOFF4: STAND-OFF, SparkFun-Electromechanical:STAND-OFF
- removed U$1: REVISION, SparkFun-Aesthetics:REVISION
- removed U1: JOYSTICKPTH, adafruit:JOYSTICKPTH
- removed U2, U5: HX711, Testing:HX711HX711
- removed U7: OSHW-LOGOS, SparkFun-Aesthetics:OSHW-LOGOS
- added 5V-2.8V-REGULATOR: (no value), v-reg:78XXS
- added JOYSTICK: JOYSTICKPTH, adafruit:JOYSTICKPTH
- added OLED-DISPLAY: (no value), SparkX:I2C_STANDARD_NO_SILK
- added R13, R14: 100K, microbuilder:RESISTOR0805_NOOUTLINE
- added R15, R16: 100K, microbuilder:RESISTOR_0805MP
- added R17: 47k, resistor-shunt:PMD
- added WIFI: (no value), microbuilder:HEADER-1X13
- C15: value (none) -> 100 nF
- C16: value (none) -> 4.7 uF
- INPUT-POWER: value AB9V -> 5 V
- R11, R12: value (none) -> 47k
- U3: value JOYSTICKPTH -> SEN-13879; device adafruit:JOYSTICKPTH -> SEN-13879:SEN-13879
- renumbered G1 to INPUT-POWER, M1 to SERVO, U4 to MICROCONTROLLER, U6 to OPTICAL-SENSOR, XTAL1 to PIEZO-BUZZER
Connections:
- removed net A+: JP4.2, JP6.2, R4.1, R7.1
- removed net A-: JP4.3, JP6.3, R3.1, R6.1
- removed net AVDD: C13.1, C3.1, C7.1, C9.1, JP4.5, JP6.5, L1.1, L2.1
- removed net B+: JP2.1, JP5.1, U2.INB+, U5.INB+
- removed net B-: JP2.2, JP5.2, U2.INB-, U5.INB-
- removed net DAT: J1.3, J2.3, MICROCONTROLLER.P4.2_A10, U2.DOUT, U5.DOUT
- removed net N$1: JP1.5, U1.H+, U1.V+
- removed net N$10: R5.1, SJ2.2, U2.RATE
- removed net N$11: C1.1, R3.2, U2.INA-
- removed net N$12: C1.2, R4.2, U2.INA+
- removed net N$2: JP1.1, U1.H-, U1.SEL-, U1.V-
- removed net N$20: C12.2, U5.VBG
- removed net N$21: L2.2, Q2.C, R9.2, U5.AVDD
- removed net N$22: R10.1, SJ1.2, U5.RATE
- removed net N$23: C10.1, R6.2, U5.INA-
- removed net N$24: C10.2, R7.2, U5.INA+
- removed net N$25: C15.2, C16.1, OPTICAL-SENSOR.AVSS_VCSEL, OPTICAL-SENSOR.GND
- removed net N$3: JP1.4, U1.V
- removed net N$4: JP1.3, U1.H
- removed net N$5: JP1.2, U1.SEL+
- removed net N$6: Q1.B, U2.BASE
- removed net N$7: R1.1, R2.2, U2.VFB
- removed net N$8: C2.2, U2.VBG
- removed net N$9: L1.2, Q1.C, R1.2, U2.AVDD
- removed net SCK: J1.4, J2.4, MICROCONTROLLER.P4.3_A11, U2.PD_SCK, U5.PD_SCK
- removed net VCC: C11.1, C5.1, C6.1, C8.1, J1.2, Q1.E, Q2.E, R10.2, R5.2, U2.VSUP, U5.VSUP
- new net !IRQ: WIFI.8
- new net +5V: 5V-2.8V-REGULATOR.IN, INPUT-POWER.+, R14.1, R16.1, WIFI.1
- new net CFG_5V: R14.2, WIFI.11
- new net CS_5V: R16.2, WIFI.6
- new net EN_5V: R15.2, WIFI.7
- new net MISO: MICROCONTROLLER.P7.3_UCB2STE_TA4.1, WIFI.4
- new net MOSI_5V: MICROCONTROLLER.P7.4__TA4.0_A16, WIFI.5
- new net N$26: MICROCONTROLLER.P4.4_TB0.5, OPTICAL-SENSOR.GPIO0, R17.2
- new net N$29: SERVO.V+
- new net RST_5V: R13.2, WIFI.9
- new net RXD_5V: WIFI.12
- new net SCK_5V: MICROCONTROLLER.P7.1_UCB2SOMI_UCB2SCL, WIFI.3
- new net SCL: OLED-DISPLAY.SCL
- new net SDA: OLED-DISPLAY.SDA
- new net TXD: WIFI.13
- new net WAKE_5V: WIFI.10
- net GND: now also 5V-2.8V-REGULATOR.GND, C15.2, C16.1, JOYSTICK.H+, JOYSTICK.H-, JOYSTICK.SEL-, JOYSTICK.V+, JOYSTICK.V-, MICROCONTROLLER.DGND, OLED-DISPLAY.GND, OPTICAL-SENSOR.AVSS_VCSEL, OPTICAL-SENSOR.GND, R13.1, R15.1, U3.GND, WIFI.2; no longer C11.2, C12.1, C13.2, C14.2, C15.1, C16.2, C2.1, C3.2, C4.2, C5.2, C6.2, C7.2, C8.2, C9.2, J1.5, J2.5, JP4.1, JP4.4, JP6.1, JP6.4, OPTICAL-SENSOR.AVDD, OPTICAL-SENSOR.AVDD_VCSEL, PIEZO-BUZZER.2, R2.1, R8.1, SERVO.V+, SJ1.1, SJ2.1, U2.AGND, U2.XI, U3.H+, U3.H-, U3.SEL-, U3.V+, U3.V-, U5.AGND, U5.XI
- net N$14: now also MICROCONTROLLER.P2.2_TB0.2_UCB0CLK, U3.CLK; no longer Q2.B, U5.BASE
- net N$15: now also JOYSTICK.V; no longer U3.V
- net N$16: now also JOYSTICK.H; no longer U3.H
- net N$17: now also JOYSTICK.SEL+; no longer U3.SEL+
- net N$19: now also MICROCONTROLLER.P2.3_TA0.0_UCA1STE_A6_C10, U3.DAT; no longer R8.2, R9.1, U5.VFB
- net VDD: now also 5V-2.8V-REGULATOR.OUT, C15.1, C16.2, MICROCONTROLLER.DVCC1, MICROCONTROLLER.P6.4_UCB3SIMO_UCB3SDA, MICROCONTROLLER.P6.6_UCB3CLK, OLED-DISPLAY.VCC, OPTICAL-SENSOR.AVDD, OPTICAL-SENSOR.AVDD_VCSEL, PIEZO-BUZZER.2, R17.1; no longer C14.1, C4.1, INPUT-POWER.+, J1.1, J2.1, J2.2, U2.DVDD, U5.DVDD
Other:
- note removed: "A+"
- note removed: "A-"
- note removed: "AVDD = VBG(R1+R2)/R1"
- note removed: "Alex Wende"
- note removed: "Black"
- note removed: "Common Load Cell Colors:"
- note removed: "Default: Closed - Data rate set to 10SPS"
- note removed: "E+"
- note removed: "E-"
- note removed: "Green or Blue"
- note removed: "IO: 2.7-5.5V"
- note removed: "N. Seidle"
- note removed: "Open jumper to set to 80SPS Increases noise per read"
- note removed: "Red"
- note removed: "Shield"
- note removed: "VBG = 1.25V"
- note removed: "VCC vs VDD: VCC is the main supply voltage, while VDD sets the digital logic voltage reference and should be connected to microcontroller supply voltage, or shorted to VCC."
- note removed: "VCC: 2.7-5.5V"
- note removed: "VDD: 2.7-5.5V"
- note removed: "White"
- note removed: "Yellow"
- note removed: "v11"
