File: Deliverable #3/Automatic Pet Feeder.brd (EAGLE design)
At the start: 38.1 x 38.1 mm, 5 parts, among them U1 JOYSTICKPTH

Commit message: Implement board
Parts:
- removed E$1: (no value), library:XTAL_PS1240P02BT_TDK
- removed E$2: (no value), library:QFN56_ESP32-S2FH4_EXP
- removed JP1: (no value), pinhead:1X05
- removed U$1: (no value), adafruit:ADAFRUIT200MIL
- removed U1: JOYSTICKPTH, adafruit:JOYSTICK
Connections:
- removed net N$1: JP1.5, U1.H1, U1.V1
- removed net N$2: JP1.1, U1.B2A, U1.H3, U1.V3
- removed net N$3: JP1.4, U1.V2
- removed net N$4: JP1.3, U1.H2
- removed net N$5: JP1.2, U1.B1A
Routing:
- net N$2: track 34.7 -> 0.00 mm
- net N$5: track 33.9 -> 0.00 mm
- net N$1: track 23.5 -> 0.00 mm
- net N$3: track 23.4 -> 0.00 mm
- net N$4: track 6.46 -> 0.00 mm
Other:
- board outline removed
- board text removed: "Analog Thumb Joystick"
- board text removed: "Breakout Board"
- board text removed: "GND"
- board text removed: "SEL shorts to ground when pressed"
- board text removed: "Sel"
- board text removed: "Vcc"
- board text removed: "X"
- board text removed: "X and Y act like 10K pots"
- board text removed: "Xout"
- board text removed: "Xout and Yout are Analog out"
- board text removed: "Y"
- board text removed: "Yout"
Changed lines of the file:
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@@
 <board>
 <plain>
-<wire x1="132.08" y1="31.75" x2="128.27" y2="35.56" width="0" layer="20" curve="90"/>
-<wire x1="128.27" y1="35.56" x2="97.79" y2="35.56" width="0" layer="20"/>
-<wire x1="97.79" y1="35.56" x2="93.98" y2="31.75" width="0" layer="20" curve="90"/>
-<wire x1="93.98" y1="31.75" x2="93.98" y2="1.27" width="0" layer="20"/>
-<wire x1="93.98" y1="1.27" x2="97.79" y2="-2.54" width="0" layer="20" curve="90"/>
-<wire x1="97.79" y1="-2.54" x2="128.27" y2="-2.54" width="0" layer="20"/>
-<wire x1="128.27" y1="-2.54" x2="132.08" y2="1.27" width="0" layer="20" curve="90"/>
-<wire x1="132.08" y1="1.27" x2="132.08" y2="31.75" width="0" layer="20"/>
-<wire x1="103.378" y1="8.636" x2="103.378" y2="3.302" width="0.3048" layer="21"/>
-<wire x1="103.378" y1="3.302" x2="102.616" y2="4.064" width="0.3048" layer="21"/>
-<wire x1="103.378" y1="3.302" x2="104.14" y2="4.064" width="0.3048" layer="21"/>
-<wire x1="102.362" y1="9.652" x2="97.028" y2="9.652" width="0.3048" layer="21"/>
-<wire x1="97.028" y1="9.652" x2="97.79" y2="8.89" width="0.3048" layer="21"/>
-<wire x1="97.028" y1="9.652" x2="97.79" y2="10.414" width="0.3048" layer="21"/>
-<text x="127.508" y="11.938" size="1.016" layer="21" font="vector" rot="R180">Vcc</text>
-<text x="128.016" y="14.478" size="1.016" layer="21" font="vector" rot="R180">Xout</text>
-<text x="128.016" y="17.018" size="1.016" layer="21" font="vector" rot="R180">Yout</text>
-<text x="127.762" y="19.558" size="1.016" layer="21" font="vector" rot="R180">Sel</text>
-<text x="127.762" y="22.098" size="1.016" layer="21" font="vector" rot="R180">GND</text>
-<text x="118.872" y="-0.254" size="1.016" layer="21" font="vector" rot="R180">Analog Thumb Joystick</text>
-<text x="118.872" y="2.032" size="1.016" layer="21" font="vector" rot="R180">Breakout Board</text>
-<text x="128.016" y="28.702" size="1.016" layer="21" font="vector" rot="R180">SEL shorts to ground when pressed</text>
-<text x="123.698" y="30.48" size="1.016" layer="21" font="vector" rot="R180">X and Y act like 10K pots</text>
-<text x="125.476" y="32.512" size="1.016" layer="21" font="vector" rot="R180">Xout and Yout are Analog out</text>
-<text x="100.33" y="8.89" size="1.778" layer="21" font="vector" rot="R180">X </text>
-<text x="102.616" y="7.112" size="1.778" layer="21" font="vector" rot="R180">Y</text>
 <hole x="128.27" y="1.27" drill="3.2"/>
 <hole x="97.79" y="1.27" drill="3.2"/>
@@
 </autorouter>
 <elements>
-<element name="E$1" library="library" package="XTAL_PS1240P02BT_TDK" value="" x="52.07" y="54.61" smashed="yes">
-<attribute name="NAME" x="51.308" y="53.975" size="1.27" layer="27" ratio="6" rot="SR0"/>
-<attribute name="VALUE" x="52.832" y="53.975" size="1.27" layer="27" ratio="6" rot="SR0"/>
-</element>
-<element name="E$2" library="library" package="QFN56_ESP32-S2FH4_EXP" value="" x="106.68" y="73.66" smashed="yes">
-<attribute name="VALUE" x="104.9528" y="73.025" size="1.27" layer="27" ratio="6" rot="SR0"/>
-</element>
-<element name="U1" library="adafruit" package="JOYSTICK" value="JOYSTICKPTH" x="113.03" y="16.51" smashed="yes" rot="R90"/>
-<element name="JP1" library="pinhead" package="1X05" value="" x="129.54" y="16.51" smashed="yes" rot="R270">
-<attribute name="VALUE" x="126.365" y="22.86" size="1.27" layer="27" rot="R270"/>
-</element>
-<element name="U$1" library="adafruit" package="ADAFRUIT200MIL" value="" x="121.158" y="0.508" smashed="yes" rot="R90"/>
 </elements>
 <signals>
-<signal name="N$1">
-<contactref element="U1" pad="V1"/>
-<contactref element="U1" pad="H1"/>
-<contactref element="JP1" pad="5"/>
-<wire x1="123.19" y1="13.716" x2="123.19" y2="13.97" width="0.4064" layer="16"/>
-<wire x1="129.54" y1="11.43" x2="125.222" y2="11.684" width="0.4064" layer="16"/>
-<wire x1="125.222" y1="11.684" x2="123.19" y2="13.716" width="0.4064" layer="16"/>
-<wire x1="110.49" y1="6.604" x2="110.49" y2="6.35" width="0.4064" layer="16"/>
-<wire x1="123.19" y1="13.97" x2="117.856" y2="13.97" width="0.4064" layer="16"/>
-<wire x1="117.856" y1="13.97" x2="110.49" y2="6.604" width="0.4064" layer="16"/>
-</signal>
-<signal name="N$2">
-<contactref element="U1" pad="V3"/>
-<contactref element="U1" pad="H3"/>
-<contactref element="U1" pad="B2A"/>
-<contactref element="JP1" pad="1"/>
-<wire x1="125.984" y1="21.844" x2="129.54" y2="21.59" width="0.4064" layer="16"/>
-<wire x1="123.19" y1="19.05" x2="125.984" y2="21.844" width="0.4064" layer="16"/>
-<wire x1="105.41" y1="13.208" x2="105.029" y2="13.335" width="0.4064" layer="1"/>
-<wire x1="115.57" y1="6.35" x2="115.57" y2="11.43" width="0.4064" layer="1"/>
-<wire x1="115.57" y1="11.43" x2="123.19" y2="19.05" width="0.4064" layer="1"/>
-<wire x1="113.792" y1="13.208" x2="105.41" y2="13.208" width="0.4064" layer="1"/>
-<wire x1="115.57" y1="11.43" x2="113.792" y2="13.208" width="0.4064" layer="1"/>
-</signal>
-<signal name="N$3">
-<contactref element="JP1" pad="4"/>
-<contactref element="U1" pad="V2"/>
-<wire x1="129.54" y1="13.97" x2="127.762" y2="14.224" width="0.4064" layer="1"/>
-<wire x1="127.762" y1="14.224" x2="117.348" y2="3.81" width="0.4064" layer="1"/>
-<wire x1="117.348" y1="3.81" x2="113.03" y2="3.81" width="0.4064" layer="1"/>
-<wire x1="113.03" y1="3.81" x2="113.03" y2="6.35" width="0.4064" layer="1"/>
-</signal>
-<signal name="N$4">
-<contactref element="JP1" pad="3"/>
-<contactref element="U1" pad="H2"/>
-<wire x1="129.54" y1="16.51" x2="123.444" y2="16.764" width="0.4064" layer="16"/>
-<wire x1="123.444" y1="16.764" x2="123.19" y2="16.51" width="0.4064" layer="16"/>
-</signal>
-<signal name="N$5">
-<contactref element="U1" pad="B1A"/>
-<contactref element="JP1" pad="2"/>
-<wire x1="103.251" y1="16.256" x2="100.529" y2="13.335" width="0.4064" layer="1"/>
-<wire x1="115.062" y1="16.256" x2="103.251" y2="16.256" width="0.4064" layer="1"/>
-<wire x1="120.904" y1="22.098" x2="115.062" y2="16.256" width="0.4064" layer="1"/>
-<wire x1="124.968" y1="22.098" x2="120.904" y2="22.098" width="0.4064" layer="1"/>
-<wire x1="127.762" y1="19.304" x2="124.968" y2="22.098" width="0.4064" layer="1"/>
-<wire x1="129.54" y1="19.05" x2="127.762" y2="19.304" width="0.4064" layer="1"/>
-</signal>
 </signals>
 <mfgpreviewcolors>
