File: Deliverable #3/Parts/Joystick (512)/Joystick-512.kicad_sch (KiCad schematic)
At the start: 2 parts, among them U1 JOYSTICKPTH

Commit message: Implement board
Parts:
- JP1: symbol joystick-eagle-import:pinhead_PINHD-1X5 -> Joystick-512:pinhead_PINHD-1X5
- U1: symbol joystick-eagle-import:adafruit_JOYSTICKPTH -> Joystick-512:adafruit_JOYSTICKPTH
Changed lines of the file:
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@@
 (kicad_sch
-	(version 20231120)
+	(version 20250114)
 	(generator "eeschema")
-	(generator_version "8.0")
+	(generator_version "9.0")
 	(paper "A4")
 	(junction
@@
 	)
 	(symbol
-		(lib_id "joystick-eagle-import:adafruit_JOYSTICKPTH")
+		(lib_id "Joystick-512:adafruit_JOYSTICKPTH")
 		(at 160.02 101.6 0)
 		(unit 1)
@@
 	)
 	(symbol
-		(lib_id "joystick-eagle-import:pinhead_PINHD-1X5")
+		(lib_id "Joystick-512:pinhead_PINHD-1X5")
 		(at 132.08 101.6 180)
 		(unit 1)
@@
 		)
 	)
+	(embedded_fonts no)
 )
