File: Deliverable #4/Automatic Pet Feeder.kicad_pcb (KiCad board)
At the start: 2 copper layers, 10 parts, among them U1 MSP430FR5994IPN, U2 TPS2513

Commit message: Added testing plan, tidied up deliverable #4 files
Parts:
- renumbered U1 to MSP430FR5994
Routing:
- net /VCC: track 280.2 -> 284.0 mm
Other:
- board text added: "0.1"
- board text added: "2025-02-27"
- board text added: "Automatic Pet Feeder"
- board text added: "CLK"
- board text added: "DAT"
- board text added: "GND"
- board text added: "PWM"
- board text added: "SCL"
- board text added: "SDA"
- board text added: "SEL"
- board text added: "Team Happy Pets Automatic Pet Feeder Sriram Vishnubhotla, Logan Swoyer"
- board text added: "VCC"
- board text added: "VDD"
- board text added: "VIN"
- board text added: "X"
- board text added: "Y"
