File: Deliverable #4/Automatic Pet Feeder.kicad_sch (KiCad schematic)
At the start: 10 parts, among them U1 MSP430FR5994IPN, U2 TPS2513

Commit message: Added testing plan, tidied up deliverable #4 files
Other:
- note added: "0.1"
- note added: "2025-02-27"
- note added: "Automatic Pet Feeder"
- note added: "Team Happy Pets Automatic Pet Feeder Sriram Vishnubhotla, Logan Swoyer"
Changed lines of the file:
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@@
 	(generator_version "9.0")
 	(paper "B")
+	(text "Team Happy Pets\nAutomatic Pet Feeder\nSriram Vishnubhotla, Logan Swoyer"
+		(exclude_from_sim no)
+		(at 313.436 243.84 0)
+		(effects
+			(font
+				(size 1.651 1.651)
+			)
+			(justify left)
+		)
+	)
+	(text "0.1"
+		(exclude_from_sim no)
+		(at 405.384 262.89 0)
+		(effects
+			(font
+				(size 1.27 1.27)
+			)
+		)
+	)
+	(text "2025-02-27"
+		(exclude_from_sim no)
+		(at 348.234 262.89 0)
+		(effects
+			(font
+				(size 1.27 1.27)
+			)
+		)
+	)
+	(text "Automatic Pet Feeder"
+		(exclude_from_sim no)
+		(at 332.232 259.08 0)
+		(effects
+			(font
+				(size 1.27 1.27)
+			)
+		)
+	)
 	(junction
 		(at 386.08 135.89)
