File: PawPlans/Hardware/PawPlans.kicad_pcb (KiCad board)
At the start: 2 copper layers, 14.2 x 21.4 mm, 5 parts

Commit message: Deliverable #6a
Connections:
- DM_PORT_A1 pad 1: unconnected-(DM_PORT_A1-SCL-Pad1) -> /SCL
- DM_PORT_A1 pad 2: unconnected-(DM_PORT_A1-SDA-Pad2) -> /SDA
- DM_PORT_B1 pad 1: unconnected-(DM_PORT_B1-IN-Pad1) -> /IN
- DM_PORT_B1 pad 2: unconnected-(DM_PORT_B1-OUT-Pad2) -> /OUT
- LD_CELL_AMP1 pad 1: unconnected-(LD_CELL_AMP1-SCL-Pad1) -> /SCL
- LD_CELL_AMP1 pad 2: unconnected-(LD_CELL_AMP1-SDA-Pad2) -> /SDA
- PROXY1 pad 1: unconnected-(PROXY1-SDA-Pad1) -> /SCL
- PROXY1 pad 2: unconnected-(PROXY1-SDA-Pad2) -> /SDA
- SERVO1 pad 1: unconnected-(SERVO1-SGN-Pad1) -> /OUT
Routing:
- net /SDA: track 0.00 -> 18.4 mm
- net /OUT: track 0.00 -> 14.5 mm
- net /SCL: track 0.00 -> 8.68 mm
Changed lines of the file:
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@@
 	)
 	(net 0 "")
-	(net 1 "unconnected-(DM_PORT_A1-SCL-Pad1)")
-	(net 2 "unconnected-(DM_PORT_A1-SDA-Pad2)")
-	(net 3 "unconnected-(DM_PORT_B1-IN-Pad1)")
-	(net 4 "unconnected-(DM_PORT_B1-OUT-Pad2)")
-	(net 5 "unconnected-(LD_CELL_AMP1-SCL-Pad1)")
-	(net 6 "unconnected-(LD_CELL_AMP1-SDA-Pad2)")
-	(net 7 "unconnected-(PROXY1-SDA-Pad1)")
-	(net 8 "unconnected-(PROXY1-SDA-Pad2)")
-	(net 9 "unconnected-(SERVO1-SGN-Pad1)")
-	(net 10 "/GND")
-	(net 11 "/5V")
+	(net 1 "/SCL")
+	(net 2 "/SDA")
+	(net 3 "/IN")
+	(net 4 "/OUT")
+	(net 5 "/GND")
+	(net 6 "/5V")
 	(footprint "Connector_PinHeader_2.54mm:PinHeader_1x04_P2.54mm_Vertical"
 		(layer "F.Cu")
@@
 			(layers "*.Cu" "*.Mask")
 			(remove_unused_layers no)
-			(net 1 "unconnected-(DM_PORT_A1-SCL-Pad1)")
+			(net 1 "/SCL")
 			(pinfunction "SCL")
 			(pintype "passive")
@@
 			(layers "*.Cu" "*.Mask")
 			(remove_unused_layers no)
-			(net 2 "unconnected-(DM_PORT_A1-SDA-Pad2)")
+			(net 2 "/SDA")
 			(pinfunction "SDA")
 			(pintype "passive")
@@
 			(layers "*.Cu" "*.Mask")
 			(remove_unused_layers no)
-			(net 11 "/5V")
+			(net 6 "/5V")
 			(pinfunction "5V")
 			(pintype "power_in")
@@
 			(layers "*.Cu" "*.Mask")
 			(remove_unused_layers no)
-			(net 10 "/GND")
+			(net 5 "/GND")
 			(pinfunction "GND")
 			(pintype "power_in")
@@
 			(layers "*.Cu" "*.Mask")
 			(remove_unused_layers no)
-			(net 3 "unconnected-(DM_PORT_B1-IN-Pad1)")
+			(net 3 "/IN")
 			(pinfunction "IN")
 			(pintype "passive")
@@
 			(layers "*.Cu" "*.Mask")
 			(remove_unused_layers no)
-			(net 4 "unconnected-(DM_PORT_B1-OUT-Pad2)")
+			(net 4 "/OUT")
 			(pinfunction "OUT")
 			(pintype "passive")
@@
 			(layers "*.Cu" "*.Mask")
 			(remove_unused_layers no)
-			(net 11 "/5V")
+			(net 6 "/5V")
 			(pinfunction "5V")
 			(pintype "power_in")
@@
 			(layers "*.Cu" "*.Mask")
 			(remove_unused_layers no)
-			(net 10 "/GND")
+			(net 5 "/GND")
 			(pinfunction "GND")
 			(pintype "power_in")
@@
 			(layers "*.Cu" "*.Mask")
 			(remove_unused_layers no)
-			(net 5 "unconnected-(LD_CELL_AMP1-SCL-Pad1)")
+			(net 1 "/SCL")
 			(pinfunction "SCL")
 			(pintype "passive")
@@
 			(layers "*.Cu" "*.Mask")
 			(remove_unused_layers no)
-			(net 6 "unconnected-(LD_CELL_AMP1-SDA-Pad2)")
+			(net 2 "/SDA")
 			(pinfunction "SDA")
 			(pintype "passive")
@@
 			(layers "*.Cu" "*.Mask")
 			(remove_unused_layers no)
-			(net 11 "/5V")
+			(net 6 "/5V")
 			(pinfunction "5V")
 			(pintype "power_in")
@@
 			(layers "*.Cu" "*.Mask")
 			(remove_unused_layers no)
-			(net 10 "/GND")
+			(net 5 "/GND")
 			(pinfunction "GND")
 			(pintype "power_in")
@@
 			(layers "*.Cu" "*.Mask")
 			(remove_unused_layers no)
-			(net 9 "unconnected-(SERVO1-SGN-Pad1)")
+			(net 4 "/OUT")
 			(pinfunction "SGN")
 			(pintype "passive")
@@
 			(layers "*.Cu" "*.Mask")
 			(remove_unused_layers no)
-			(net 11 "/5V")
+			(net 6 "/5V")
 			(pinfunction "5V")
 			(pintype "passive")
@@
 			(layers "*.Cu" "*.Mask")
 			(remove_unused_layers no)
-			(net 10 "/GND")
+			(net 5 "/GND")
 			(pinfunction "GND")
 			(pintype "power_in")
@@
 			(layers "*.Cu" "*.Mask")
 			(remove_unused_layers no)
-			(net 7 "unconnected-(PROXY1-SDA-Pad1)")
+			(net 1 "/SCL")
 			(pinfunction "SDA")
 			(pintype "passive")
@@
 			(layers "*.Cu" "*.Mask")
 			(remove_unused_layers no)
-			(net 8 "unconnected-(PROXY1-SDA-Pad2)")
+			(net 2 "/SDA")
 			(pinfunction "SDA")
 			(pintype "passive")
@@
 			(layers "*.Cu" "*.Mask")
 			(remove_unused_layers no)
-			(net 11 "/5V")
+			(net 6 "/5V")
 			(pinfunction "5V")
 			(pintype "power_in")
@@
 			(layers "*.Cu" "*.Mask")
 			(remove_unused_layers no)
-			(net 10 "/GND")
+			(net 5 "/GND")
 			(pinfunction "GND")
 			(pintype "power_in")
@@
 		)
 	)
+	(segment
+		(start 100 63.65)
+		(end 100 67.525)
+		(width 0.2)
+		(layer "F.Cu")
+		(net 1)
+	)
+	(segment
+		(start 100 67.525)
+		(end 104.8 67.525)
+		(width 0.2)
+		(layer "F.Cu")
+		(net 1)
+	)
+	(segment
+		(start 100 70.065)
+		(end 104.8 70.065)
+		(width 0.2)
+		(layer "F.Cu")
+		(net 2)
+	)
+	(segment
+		(start 102.54 63.65)
+		(end 100.89 62)
+		(width 0.2)
+		(layer "F.Cu")
+		(net 2)
+	)
+	(segment
+		(start 100.89 62)
+		(end 98.4 62)
+		(width 0.2)
+		(layer "F.Cu")
+		(net 2)
+	)
+	(segment
+		(start 98.4 68.465)
+		(end 100 70.065)
+		(width 0.2)
+		(layer "F.Cu")
+		(net 2)
+	)
+	(segment
+		(start 98.4 62)
+		(end 98.4 68.465)
+		(width 0.2)
+		(layer "F.Cu")
+		(net 2)
+	)
+	(segment
+		(start 102.54 59)
+		(end 105.54 62)
+		(width 0.2)
+		(layer "F.Cu")
+		(net 4)
+	)
+	(segment
+		(start 109.4 68.4)
+		(end 109 68.8)
+		(width 0.2)
+		(layer "F.Cu")
+		(net 4)
+	)
+	(segment
+		(start 105.54 62)
+		(end 108.4 62)
+		(width 0.2)
+		(layer "F.Cu")
+		(net 4)
+	)
+	(segment
+		(start 108.4 62)
+		(end 109.4 63)
+		(width 0.2)
+		(layer "F.Cu")
+		(net 4)
+	)
+	(segment
+		(start 109.4 63)
+		(end 109.4 68.4)
+		(width 0.2)
+		(layer "F.Cu")
+		(net 4)
+	)
 	(zone
-		(net 11)
+		(net 6)
 		(net_name "/5V")
 		(layer "F.Cu")
@@
 	)
 	(zone
-		(net 10)
+		(net 5)
 		(net_name "/GND")
 		(layer "B.Cu")
