File: PawPlans/Hardware/PawPlans.kicad_sch (KiCad schematic)
At the start: 5 parts

Commit message: Deliverable #6a
Connections:
- net IN: now reaches DM_PORT_B1.1 (IN)
- net OUT: now reaches DM_PORT_B1.2 (OUT)
- net OUT: now also SERVO1.1 (SGN)
- net SCL: now reaches PROXY1.1 (SDA)
- net SCL: now also DM_PORT_A1.1 (SCL), LD_CELL_AMP1.1 (SCL)
- net SDA: now reaches PROXY1.2 (SDA)
- net SDA: now also DM_PORT_A1.2 (SDA), LD_CELL_AMP1.2 (SDA)
Changed lines of the file:
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@@
+	(wire
+		(pts
+			(xy 116.84 60.96) (xy 119.38 60.96)
+		)
+		(stroke
+			(width 0)
+			(type default)
+		)
+	)
 	(wire
 		(pts
@@
 	(wire
 		(pts
+			(xy 93.98 60.96) (xy 96.52 60.96)
+		)
+		(stroke
+			(width 0)
+			(type default)
+		)
+	)
+	(wire
+		(pts
+			(xy 138.43 62.23) (xy 140.97 62.23)
+		)
+		(stroke
+			(width 0)
+			(type default)
+		)
+	)
+	(wire
+		(pts
+			(xy 76.2 63.5) (xy 78.74 63.5)
+		)
+		(stroke
+			(width 0)
+			(type default)
+		)
+	)
+	(wire
+		(pts
+			(xy 93.98 63.5) (xy 96.52 63.5)
+		)
+		(stroke
+			(width 0)
+			(type default)
+		)
+	)
+	(wire
+		(pts
+			(xy 54.61 63.5) (xy 57.15 63.5)
+		)
+		(stroke
+			(width 0)
+			(type default)
+		)
+	)
+	(wire
+		(pts
 			(xy 76.2 66.04) (xy 78.74 66.04)
 		)
@@
 	(wire
 		(pts
+			(xy 54.61 60.96) (xy 57.15 60.96)
+		)
+		(stroke
+			(width 0)
+			(type default)
+		)
+	)
+	(wire
+		(pts
 			(xy 138.43 67.31) (xy 140.97 67.31)
 		)
@@
 	(wire
 		(pts
+			(xy 76.2 60.96) (xy 78.74 60.96)
+		)
+		(stroke
+			(width 0)
+			(type default)
+		)
+	)
+	(wire
+		(pts
 			(xy 93.98 66.04) (xy 96.52 66.04)
 		)
@@
 		)
 	)
+	(wire
+		(pts
+			(xy 116.84 63.5) (xy 119.38 63.5)
+		)
+		(stroke
+			(width 0)
+			(type default)
+		)
+	)
 	(label "GND"
 		(at 116.84 68.58 180)
@@
 		)
 	)
+	(label "SCL"
+		(at 116.84 60.96 180)
+		(effects
+			(font
+				(size 1.27 1.27)
+			)
+			(justify right bottom)
+		)
+	)
 	(label "5V"
 		(at 116.84 66.04 180)
@@
 		)
 	)
+	(label "SDA"
+		(at 93.98 63.5 180)
+		(effects
+			(font
+				(size 1.27 1.27)
+			)
+			(justify right bottom)
+		)
+	)
 	(label "5V"
 		(at 138.43 64.77 180)
@@
 		)
 	)
+	(label "SCL"
+		(at 93.98 60.96 180)
+		(effects
+			(font
+				(size 1.27 1.27)
+			)
+			(justify right bottom)
+		)
+	)
 	(label "GND"
 		(at 93.98 68.58 180)
@@
 		)
 	)
+	(label "SCL"
+		(at 54.61 60.96 180)
+		(effects
+			(font
+				(size 1.27 1.27)
+			)
+			(justify right bottom)
+		)
+	)
+	(label "OUT"
+		(at 76.2 63.5 180)
+		(effects
+			(font
+				(size 1.27 1.27)
+			)
+			(justify right bottom)
+		)
+	)
+	(label "SDA"
+		(at 54.61 63.5 180)
+		(effects
+			(font
+				(size 1.27 1.27)
+			)
+			(justify right bottom)
+		)
+	)
 	(label "GND"
 		(at 54.61 68.58 180)
@@
 		)
 	)
+	(label "IN"
+		(at 76.2 60.96 180)
+		(effects
+			(font
+				(size 1.27 1.27)
+			)
+			(justify right bottom)
+		)
+	)
 	(label "5V"
 		(at 76.2 66.04 180)
@@
 		(effects
 			(font
+				(size 1.27 1.27)
+			)
+			(justify right bottom)
+		)
+	)
+	(label "SDA"
+		(at 116.84 63.5 180)
+		(effects
+			(font
+				(size 1.27 1.27)
+			)
+			(justify right bottom)
+		)
+	)
+	(label "OUT"
+		(at 138.43 62.23 180)
+		(effects
+			(font
